Commit message: added fancy wheels
and changed fixed frame of rviz config file to base_footprint

File: urdf/youbot_base/base.urdf.xacro (robot description, xacro)
@@ -4,4 +4,5 @@
        xmlns:interface="http://playerstage.sourceforge.net/gazebo/xmlschema/#interface"
        xmlns:xacro="http://ros.org/wiki/xacro">
+  <!-- sensors -->
   <xacro:include filename="$(find youbot_description)/urdf/youbot_base/base.gazebo.xacro"/>
   <xacro:include filename="$(find youbot_description)/urdf/youbot_base/base.transmission.xacro"/>
@@ -32,4 +33,27 @@
   <property name="wheel_joint_safety_k_velocity" value="10.0"/>
   <xacro:macro name="youbot_base" params="name">
+<!--     <link name="odom" />
+    <joint name="base_x_joint" type="prismatic">
+      <origin xyz="0 0 0.07" rpy="0 0 0"/>
+      <limit effort="10.0" lower="-5.0" upper="5.0" velocity="0.1"/>
+      <child link="dummy_link_x"/>
+      <parent link="odom"/>
+    </joint>
+    <link name="dummy_link_x" />
+    <joint name="base_y_joint" type="prismatic">
+      <origin xyz="0 0 0" rpy="0 0 0"/>
+      <limit effort="10.0" lower="-5.0" upper="5.0" velocity="0.1"/>
+      <axis xyz="0 1 0"/>
+      <child link="dummy_link_y"/>
+      <parent link="dummy_link_x"/>
+    </joint>
+    <link name="dummy_link_y" />
+    <joint name="base_rotational_joint" type="continuous">
+      <origin xyz="0 0 0" rpy="0 0 0"/>
+      <limit effort="10.0" velocity="0.1"/>
+      <axis xyz="0 0 1"/>
+      <child link="base_link"/>
+      <parent link="dummy_link_y"/>
+    </joint> -->
     <link name="${name}_footprint">
       <inertial>
@@ -43,5 +67,5 @@
           <box size="0.001 0.001 0.001"/>
         </geometry>
-        <material name="youBot/Red"/>
+        <material name="Red"/>
       </visual>
       <collision>
@@ -68,5 +92,5 @@
           <mesh filename="package://youbot_description/meshes/youbot_base/base.dae"/>
         </geometry>
-        <material name="youBot/DarkGrey"/>
+        <material name="DarkGrey"/>
       </visual>
       <collision>
@@ -79,5 +103,5 @@
     </link>
     <!-- front left wheel -->
-    <joint name="caster_joint_fl" type="continuous">
+    <joint name="caster_joint_fl" type="fixed">
       <origin xyz="${caster_offset_x} ${caster_offset_y} ${caster_offset_z}" rpy="0 0 0"/>
       <axis xyz="0 0 1"/>
@@ -114,7 +138,7 @@
         <!--<mesh filename="package://youbot_description/meshes/youbot_base/youbot_wheel.stl" />-->
         <geometry>
-          <sphere radius="${wheel_radius}"/>
-        </geometry>
-        <material name="youBot/Orange"/>
+          <mesh filename="package://youbot_description/meshes/youbot_base/front-left_wheel.dae" />
+        </geometry>
+        <material name="Orange"/>
       </visual>
       <collision>
@@ -126,5 +150,5 @@
     </link>
     <!-- front right wheel -->
-    <joint name="caster_joint_fr" type="continuous">
+    <joint name="caster_joint_fr" type="fixed">
       <origin xyz="${caster_offset_x} ${-caster_offset_y} ${caster_offset_z}" rpy="0 0 0"/>
       <axis xyz="0 0 1"/>
@@ -161,7 +185,7 @@
         <geometry>
           <!--<mesh filename="package://youbot_description/meshes/youbot_base/youbot_wheel.stl" />-->
-          <sphere radius="${wheel_radius}"/>
-        </geometry>
-        <material name="youBot/Orange"/>
+          <mesh filename="package://youbot_description/meshes/youbot_base/front-right_wheel.dae" />
+        </geometry>
+        <material name="Orange"/>
       </visual>
       <collision>
@@ -173,5 +197,5 @@
     </link>
     <!-- back left wheel -->
-    <joint name="caster_joint_bl" type="continuous">
+    <joint name="caster_joint_bl" type="fixed">
       <origin xyz="${-caster_offset_x} ${caster_offset_y} ${caster_offset_z}" rpy="0 0 0"/>
       <axis xyz="0 0 1"/>
@@ -209,7 +233,7 @@
         <geometry>
           <!--<mesh filename="package://youbot_description/meshes/youbot_base/youbot_wheel.stl" />-->
-          <sphere radius="${wheel_radius}"/>
-        </geometry>
-        <material name="youBot/Orange"/>
+          <mesh filename="package://youbot_description/meshes/youbot_base/back-left_wheel.dae" />
+        </geometry>
+        <material name="Orange"/>
       </visual>
       <collision>
@@ -221,5 +245,5 @@
     </link>
     <!-- back right wheel -->
-    <joint name="caster_joint_br" type="continuous">
+    <joint name="caster_joint_br" type="fixed">
       <origin xyz="${-caster_offset_x} ${-caster_offset_y} ${caster_offset_z}" rpy="0 0 0"/>
       <axis xyz="0 0 1"/>
@@ -256,7 +280,7 @@
         <geometry>
           <!--<mesh filename="package://youbot_description/meshes/youbot_base/youbot_wheel.stl" />-->
-          <sphere radius="${wheel_radius}"/>
-        </geometry>
-        <material name="youBot/Orange"/>
+          <mesh filename="package://youbot_description/meshes/youbot_base/back-right_wheel.dae" />
+        </geometry>
+        <material name="Orange"/>
       </visual>
       <collision>
