Commit message: flipped the laser scanner and added the xtion to gripper_palm_link

File: robots/youbot.urdf.xacro (robot description, xacro)
@@ -22,4 +22,5 @@
   <!-- sensors -->
   <xacro:include filename="$(find youbot_description)/urdf/sensors/hokuyo_urg04_laser.urdf.xacro"/>
+  <xacro:include filename="$(find youbot_description)/urdf/sensors/asus_xtion_camera.urdf.xacro"/>
   <!-- Now we can start using the macros xacro:included above to define the actual youbot -->
   <!-- The first use of a macro.  This one was defined in base.urdf.xacro above.
@@ -42,6 +43,9 @@
   </xacro:youbot_gripper>
   <!-- base laser front -->
-  <xacro:hokuyo_urg04_laser name="base_laser_front" parent="base" ros_topic="scan_front" update_rate="10" min_angle="-1.57" max_angle="1.57">
-    <origin xyz="0.3 0 -0.03" rpy="0 0 0"/>
+  <xacro:hokuyo_urg04_laser name="base_laser_front" parent="base" ros_topic="base_scan" update_rate="10" min_angle="-1.57" max_angle="1.57">
+    <origin xyz="0.3 0 -0.03" rpy="3.14 0 0"/>
   </xacro:hokuyo_urg04_laser>
+  <xacro:asus_xtion_camera name="xtion" parent="gripper_palm_link" tilt="0.0">
+    <origin xyz="0.025 0.0 -0.032" rpy="3.14 -1.6 0.0" />
+  </xacro:asus_xtion_camera>
 </robot>
